Commit message: ackermann vehicle controller basic structure, gazebo friction tags in urdf, ros2_control controller setup

File: model/f1tenth_model.urdf.xacro (robot description, xacro)
@@ -16,5 +16,8 @@
     <xacro:property name="knuckle_mass" value="${arm_mass * (arm_length - knuckle_radius) / arm_length}" />
     <xacro:property name="max_steering_angle" value="0.36" />
-    <xacro:property name="max_steering_velocity" value="2.0" />
+    <xacro:property name="max_steering_angular_velocity" value="2.0" />
+    <xacro:property name="max_wheel_angular_velocity" value="20.0"/>
+    <xacro:property name="wheel_mu" value="1.5" />
+    <xacro:property name="chassis_mu" value="0.1" />
     <material name="papaya orange">
         <color rgba="1.0 ${128 / 255} 0.0 1.0" />
@@ -209,5 +212,18 @@
     </ros2_control>
     <gazebo>
-        <plugin filename="libgz_ros2_control-system.so" name="gz_ros2_control::GazeboSimROS2ControlPlugin" />
+        <plugin filename="libgz_ros2_control-system.so" name="gz_ros2_control::GazeboSimROS2ControlPlugin">
+            <parameters>$(find f1tenth_gz_sim)/config/vehicle_controllers.yaml</parameters>
+        </plugin>
     </gazebo>
+    <xacro:macro name="gz_friction" params="link mu">
+        <gazebo reference="${link}">
+            <mu1>${mu}</mu1>
+            <mu2>${mu}</mu2>
+        </gazebo>
+    </xacro:macro>
+    <xacro:gz_friction link="front_left_wheel" mu="${wheel_mu)" />
+    <xacro:gz_friction link="front_right_wheel" mu="${wheel_mu)" />
+    <xacro:gz_friction link="back_left_wheel" mu="${wheel_mu)" />
+    <xacro:gz_friction link="back_right_wheel" mu="${wheel_mu)" />
+    <xacro:gz_friction link="chassis" mu="${chassis_mu)" />
 </robot>

Commit message: added bridge for sim time, tested with a message (it moves)

File: model/f1tenth_model.urdf.xacro (robot description, xacro)
@@ -166,5 +166,5 @@
             <child link="${prefix}_steering_knuckle" />
             <axis xyz="0 0 1" />
-            <limit lower="${-max_steering_angle}" upper="${max_steering_angle}" effort="10.0" velocity="${max_steering_velocity}"/>
+            <limit lower="${-max_steering_angle}" upper="${max_steering_angle}" effort="10.0" velocity="${max_steering_angular_velocity}"/>
             <origin xyz="0 ${y_offset} 0" rpy="0 0 0" />
         </joint>
@@ -195,7 +195,13 @@
         </joint>
     </xacro:macro>
+    <xacro:macro name="ros2_control_cmd_spinning" params="prefix">
+        <joint name="${prefix}_spinning">
+            <command_interface name="velocity" />
+            <state_interface name="velocity"/>
+            <state_interface name="position"/>
+        </joint>
+    </xacro:macro>
     <xacro:macro name="ros2_control_spinning" params="prefix">
         <joint name="${prefix}_spinning">
-            <command_interface  name="velocity" />
             <state_interface name="velocity"/>
             <state_interface name="position"/>
@@ -208,6 +214,8 @@
         <xacro:ros2_control_steering prefix="front_left" max_angle="${max_steering_angle}"/>
         <xacro:ros2_control_steering prefix="front_right" max_angle="${max_steering_angle}"/>
-        <xacro:ros2_control_spinning prefix="back_left"/>
-        <xacro:ros2_control_spinning prefix="back_right"/>
+        <xacro:ros2_control_spinning prefix="front_left"/>
+        <xacro:ros2_control_spinning prefix="front_right"/>
+        <xacro:ros2_control_cmd_spinning prefix="back_left"/>
+        <xacro:ros2_control_cmd_spinning prefix="back_right"/>
     </ros2_control>
     <gazebo>
@@ -222,8 +230,8 @@
         </gazebo>
     </xacro:macro>
-    <xacro:gz_friction link="front_left_wheel" mu="${wheel_mu)" />
-    <xacro:gz_friction link="front_right_wheel" mu="${wheel_mu)" />
-    <xacro:gz_friction link="back_left_wheel" mu="${wheel_mu)" />
-    <xacro:gz_friction link="back_right_wheel" mu="${wheel_mu)" />
-    <xacro:gz_friction link="chassis" mu="${chassis_mu)" />
+    <xacro:gz_friction link="front_left_wheel" mu="${wheel_mu}" />
+    <xacro:gz_friction link="front_right_wheel" mu="${wheel_mu}" />
+    <xacro:gz_friction link="back_left_wheel" mu="${wheel_mu}" />
+    <xacro:gz_friction link="back_right_wheel" mu="${wheel_mu}" />
+    <xacro:gz_friction link="chassis" mu="${chassis_mu}" />
 </robot>

Commit message: tweaked model, added ackermann steering calcs, parameters, switch to 4WD

File: model/f1tenth_model.urdf.xacro (robot description, xacro)
@@ -10,10 +10,10 @@
     <xacro:property name="wheel_length" value="0.04318" />
     <xacro:property name="tire_thickness" value="0.012" />
-    <xacro:property name="arm_length" value="0.012" />
+    <xacro:property name="arm_length" value="0.019" />
     <xacro:property name="arm_radius" value="0.005" />
     <xacro:property name="arm_mass" value="0.005" />
     <xacro:property name="knuckle_radius" value="0.0025" />
     <xacro:property name="knuckle_mass" value="${arm_mass * (arm_length - knuckle_radius) / arm_length}" />
-    <xacro:property name="max_steering_angle" value="0.36" />
+    <xacro:property name="max_steering_angle" value="0.6" />
     <xacro:property name="max_steering_angular_velocity" value="2.0" />
     <xacro:property name="max_wheel_angular_velocity" value="20.0"/>
@@ -157,8 +157,8 @@
     </xacro:macro>
     <!-- Wheel Spinning joint definition -->
-    <xacro:spinning_joint prefix="front_left" parent="steering_knuckle" y_offset="${-(knuckle_radius + wheel_length / 2)}" />
-    <xacro:spinning_joint prefix="front_right" parent="steering_knuckle" y_offset="${knuckle_radius + wheel_length / 2}" />
-    <xacro:spinning_joint prefix="back_left" parent="arm" y_offset="${-(arm_length / 2 + wheel_length / 2)}" />
-    <xacro:spinning_joint prefix="back_right" parent="arm" y_offset="${arm_length / 2 + wheel_length / 2}" />
+    <xacro:spinning_joint prefix="front_right" parent="steering_knuckle" y_offset="${-(knuckle_radius + wheel_length / 2)}" />
+    <xacro:spinning_joint prefix="front_left" parent="steering_knuckle" y_offset="${knuckle_radius + wheel_length / 2}" />
+    <xacro:spinning_joint prefix="back_right" parent="arm" y_offset="${-(arm_length / 2 + wheel_length / 2)}" />
+    <xacro:spinning_joint prefix="back_left" parent="arm" y_offset="${arm_length / 2 + wheel_length / 2}" />
     <xacro:macro name="steering_joint" params="prefix y_offset" >
         <joint name="${prefix}_steering" type="revolute">
@@ -171,6 +171,6 @@
     </xacro:macro>
     <!-- Steering joint definitions -->
-    <xacro:steering_joint prefix="front_left" y_offset="${-((arm_length - knuckle_radius) / 2 + knuckle_radius)}" />
-    <xacro:steering_joint prefix="front_right" y_offset="${(arm_length - knuckle_radius) / 2 + knuckle_radius}" />
+    <xacro:steering_joint prefix="front_right" y_offset="${-((arm_length - knuckle_radius) / 2 + knuckle_radius)}" />
+    <xacro:steering_joint prefix="front_left" y_offset="${(arm_length - knuckle_radius) / 2 + knuckle_radius}" />
     <xacro:macro name="arm_joint" params="prefix x_offset y_offset" >
         <joint name="${prefix}_arm_fixed" type="fixed">
@@ -181,8 +181,8 @@
     </xacro:macro>
     <!-- Arm to chassis joints -->
-    <xacro:arm_joint prefix="front_left" x_offset="${wheelbase / 2}" y_offset="${-((arm_length - knuckle_radius) / 2 + chassis_width / 2)}" />
-    <xacro:arm_joint prefix="front_right" x_offset="${wheelbase / 2}" y_offset="${(arm_length - knuckle_radius) / 2 + chassis_width / 2}" />
-    <xacro:arm_joint prefix="back_left" x_offset="${-wheelbase / 2}" y_offset="${-(arm_length / 2 + chassis_width / 2)}" />
-    <xacro:arm_joint prefix="back_right" x_offset="${-wheelbase / 2}" y_offset="${arm_length / 2 + chassis_width / 2}" />
+    <xacro:arm_joint prefix="front_right" x_offset="${wheelbase / 2}" y_offset="${-((arm_length - knuckle_radius) / 2 + chassis_width / 2)}" />
+    <xacro:arm_joint prefix="front_left" x_offset="${wheelbase / 2}" y_offset="${(arm_length - knuckle_radius) / 2 + chassis_width / 2}" />
+    <xacro:arm_joint prefix="back_right" x_offset="${-wheelbase / 2}" y_offset="${-(arm_length / 2 + chassis_width / 2)}" />
+    <xacro:arm_joint prefix="back_left" x_offset="${-wheelbase / 2}" y_offset="${arm_length / 2 + chassis_width / 2}" />
     <xacro:macro name="ros2_control_steering" params="prefix max_angle">
         <joint name="${prefix}_steering">
@@ -195,13 +195,7 @@
         </joint>
     </xacro:macro>
-    <xacro:macro name="ros2_control_cmd_spinning" params="prefix">
+    <xacro:macro name="ros2_control_spinning" params="prefix">
         <joint name="${prefix}_spinning">
             <command_interface name="velocity" />
-            <state_interface name="velocity"/>
-            <state_interface name="position"/>
-        </joint>
-    </xacro:macro>
-    <xacro:macro name="ros2_control_spinning" params="prefix">
-        <joint name="${prefix}_spinning">
             <state_interface name="velocity"/>
             <state_interface name="position"/>
@@ -216,6 +210,6 @@
         <xacro:ros2_control_spinning prefix="front_left"/>
         <xacro:ros2_control_spinning prefix="front_right"/>
-        <xacro:ros2_control_cmd_spinning prefix="back_left"/>
-        <xacro:ros2_control_cmd_spinning prefix="back_right"/>
+        <xacro:ros2_control_spinning prefix="back_left"/>
+        <xacro:ros2_control_spinning prefix="back_right"/>
     </ros2_control>
     <gazebo>
@@ -223,4 +217,12 @@
             <parameters>$(find f1tenth_gz_sim)/config/vehicle_controllers.yaml</parameters>
         </plugin>
+        <!-- <plugin filename="gz-sim-imu-system"
+            name="gz::sim::systems::Imu">
+        </plugin>
+        <plugin
+            filename="gz-sim-sensors-system"
+            name="gz::sim::systems::Sensors">
+            <render_engine>ogre2</render_engine>
+        </plugin> -->
     </gazebo>
     <xacro:macro name="gz_friction" params="link mu">
