Commit message: added lidar

File: model/f1tenth_car.urdf.xacro (robot description, xacro)
@@ -38,14 +38,18 @@
     <xacro:property name="max_wheel_angular_velocity" value="$(arg max_wheel_angular_velocity)"/>
     <xacro:property name="knuckle_mass" value="${arm_mass * (arm_length - 2 * knuckle_radius) / arm_length}" />
+    <xacro:property name="lidar_radius" value="0.053"/>
+    <xacro:property name="lidar_length" value="0.087"/>
+    <xacro:property name="lidar_mass" value="0.37" />
+    <xacro:property name="lidar_angle" value="${radians(135)}"/>
     <material name="papaya orange">
         <color rgba="1.0 ${128 / 255} 0.0 1.0" />
     </material>
-    <material name="tire color">
+    <material name="black">
         <color rgba="0.0 0.0 0.0 1.0" />
     </material>
-    <material name="steering link color">
+    <material name="red-orange">
         <color rgba="${189 / 255} ${55 / 255} ${10 / 255} 1.0" />
     </material>
-    <material name="steering arm color">
+    <material name="grey">
         <color rgba="${166 / 255} ${166 / 255} ${166 / 255} 1.0" />
     </material>
@@ -72,5 +76,5 @@
         <visual>
             <geometry>
-                <box size="${chassis_length} ${chassis_width} ${chassis_height}"/>
+                <box size="${chassis_length} ${chassis_width + 2 * arm_length} ${chassis_height}"/>
             </geometry>
             <material name="papaya orange" />
@@ -96,5 +100,5 @@
             <visual>
                 <xacro:cylinder_geometry length="${length}" radius="${radius}" />
-                <material name="tire color"/>
+                <material name="black"/>
                 <origin xyz="0 0 0" rpy="${pi/2} 0 0" />
             </visual>
@@ -120,9 +124,17 @@
         </inertial>
     </xacro:macro>
+    <xacro:macro name="cylinder_inertial" params="mass radius length">
+        <inertial>
+            <mass value="${mass}" />
+            <inertia ixx="${1 / 12 * mass * (3 * radius * radius + length * length)}" ixy="0.0" ixz="0.0"
+                        iyy="${1 / 12 * mass * (3 * radius * radius + length * length)}" iyz="0.0"
+                        izz="${1 / 2 * mass * radius * radius}" />
+        </inertial>
+    </xacro:macro>
     <xacro:macro name="arm" params="prefix mass radius length">
         <link name="${prefix}_arm">
             <visual>
                 <xacro:cylinder_geometry length="${length}" radius="${radius}" />
-                <material name="steering arm color"/>
+                <material name="grey"/>
                 <origin xyz="0 0 0" rpy="${pi/2} 0 0" />
             </visual>
@@ -153,5 +165,5 @@
                     <sphere radius="${radius}"/>
                 </geometry>
-                <material name="steering link color"/>
+                <material name="red-orange"/>
             </visual>
             <collision>
@@ -213,5 +225,5 @@
         </joint>
     </xacro:macro>
-    <xacro:macro name="ros2_control_spinning" params="prefix">
+   <xacro:macro name="ros2_control_spinning" params="prefix">
         <joint name="${prefix}_spinning">
             <command_interface name="velocity" />
@@ -220,5 +232,5 @@
         </joint>
     </xacro:macro>
-    <ros2_control name="GazeboSimSystem" type="system">
+    <ros2_control name="f1tenth_car_control" type="system">
         <hardware>
             <plugin>gz_ros2_control/GazeboSimSystem</plugin>
@@ -235,11 +247,11 @@
             <parameters>$(find f1tenth_gz_sim)/config/vehicle_controllers.yaml</parameters>
         </plugin>
-        <!-- <plugin filename="gz-sim-imu-system"
-            name="gz::sim::systems::Imu">
-        </plugin>
         <plugin
             filename="gz-sim-sensors-system"
             name="gz::sim::systems::Sensors">
             <render_engine>ogre2</render_engine>
+        </plugin>
+        <!-- <plugin filename="gz-sim-imu-system"
+            name="gz::sim::systems::Imu">
         </plugin> -->
     </gazebo>
@@ -255,3 +267,46 @@
     <xacro:gz_friction link="back_right_wheel" mu="${wheel_mu}" />
     <xacro:gz_friction link="chassis" mu="${chassis_mu}" />
+        <!-- hokuyo lidar (UTM - 30LX) -->
+    <link name="laser_frame">
+        <collision>
+            <geometry>
+                <cylinder length="${lidar_length}" radius="${lidar_radius}"/>
+            </geometry>
+        </collision>
+        <visual>
+            <geometry>
+                <cylinder length="${lidar_length}" radius="${lidar_radius}"/>
+            </geometry>
+            <material name="black" />
+        </visual>
+        <xacro:cylinder_inertial mass="${lidar_mass}" radius="${lidar_radius}" length="${lidar_length}"/>
+    </link>
+    <joint name="laser_joint" type="fixed" >
+        <parent link="chassis" />
+        <child link="laser_frame" />
+        <origin xyz="0.14 0 ${chassis_height/2 + lidar_length / 2}" rpy="0 0 0" />
+    </joint>
+    <gazebo reference="laser_frame">
+        <sensor name="hokuyo_lidar" type="gpu_lidar">
+            <topic>/scan</topic>
+            <pose relative_to="laser_frame"> 0 0 0 0 0 0</pose>
+            <visualize>true</visualize>
+            <always_on>true</always_on>
+            <update_rate>20</update_rate>
+            <lidar>
+                <scan>
+                    <horizontal>
+                        <samples>1440</samples>
+                        <min_angle>${-(lidar_angle)}</min_angle>
+                        <max_angle>${lidar_angle}</max_angle>
+                    </horizontal>
+                </scan>
+                <range>
+                    <min>0.1</min>
+                    <max>30</max>
+                    <resolution>0.01</resolution>
+                </range>
+            </lidar>
+        </sensor>
+    </gazebo>
 </robot>
